Commit message: [add]controller

File: Robot_2D_navigation/xacro/robot.xacro (robot description, xacro)
@@ -82,5 +82,5 @@
   </link>
   <gazebo reference="body_link">
-    <material>Gazebo/Gray</material>
+    <material>Gazebo/White</material>
   </gazebo>
   <xacro:wheel_macro prefix="left_wheel"  parent="base_link" xyz="0 0.1 0.05"/>
